Commit message: scara config has urdf issues. default urdf is working fine.

File: src/scara_4dof/urdf/scara_controller/robot_controller.ros2_control.xacro (robot description, xacro)
@@ -1,5 +1,5 @@
 <?xml version="1.0"?>
 <robot xmlns:xacro="http://www.ros.org/wiki/xacro">
-    <xacro:macro name="scara_control_control" params="
+    <xacro:macro name="robot_control_control" params="
       name
       prefix
@@ -14,7 +14,7 @@
               <param name="master_config">${master_config}</param>
               <param name="can_interface_name">${can_interface_name}</param>
-              <param name="master_bin">${master_bin}</param>
+              <param name="master_bin">"${master_bin}"</param>
             </hardware>
-            <!-- Prismatic joint configuration -->
+            <!-- Prismatic Joint -->
             <joint name="${prefix}joint1">
                 <param name="device_name">joint_1</param>
@@ -22,21 +22,25 @@
                 <command_interface name="position" />
             </joint>
-            <!-- Revolute joint 1 configuration -->
+            <!-- Revolute Joints -->
             <joint name="${prefix}joint2">
                 <param name="device_name">joint_2</param>
                 <state_interface name="position" />
                 <command_interface name="position" />
+                <state_interface name="velocity" />
+                <command_interface name="velocity" />
             </joint>
-            <!-- Revolute joint 2 configuration -->
             <joint name="${prefix}joint3">
                 <param name="device_name">joint_3</param>
                 <state_interface name="position" />
                 <command_interface name="position" />
+                <state_interface name="velocity" />
+                <command_interface name="velocity" />
             </joint>
-            <!-- Revolute joint 3 configuration -->
             <joint name="${prefix}joint4">
                 <param name="device_name">joint_4</param>
                 <state_interface name="position" />
                 <command_interface name="position" />
+                <state_interface name="velocity" />
+                <command_interface name="velocity" />
             </joint>
         </ros2_control>
