Commit message: four joint controller is working successfully.

File: src/scara_4dof/urdf/robot_controller/robot_controller.macro.xacro (robot description, xacro)
@@ -44,5 +44,5 @@
         <child link="${prefix}link1"/>
     </joint>
-    <joint name="${prefix}joint1" type="revolute">
+    <joint name="${prefix}joint1" type="prismatic">
         <parent link="${prefix}link1"/>
         <child link="${prefix}link2"/>

File: src/scara_4dof/urdf/robot_controller/robot_controller.urdf.xacro (robot description, xacro)
@@ -1,6 +1,6 @@
 <?xml version="1.0"?>
 <robot xmlns:xacro="http://wiki.ros.org/xacro" name="test_robot">
-    <xacro:include filename="$(find canopen_tests)/urdf/robot_controller/robot_controller.macro.xacro"/>
-    <xacro:include filename="$(find canopen_tests)/urdf/robot_controller/robot_controller.ros2_control.xacro"/>
+    <xacro:include filename="$(find scara_4dof)/urdf/scara_controller/robot_controller.macro.xacro"/>
+    <xacro:include filename="$(find scara_4dof)/urdf/scara_controller/robot_controller.ros2_control.xacro"/>
     <link name="world" />
     <xacro:robot_control_robot
@@ -14,6 +14,6 @@
         name="test_robot"
         prefix=""
-        bus_config="$(find canopen_tests)/config/robot_control/bus.yml"
-        master_config="$(find canopen_tests)/config/robot_control/master.dcf"
+        bus_config="$(find canopen_tests)/config/scara_4dof_control/bus.yml"
+        master_config="$(find canopen_tests)/config/scara_4dof_control/master.dcf"
         can_interface_name="vcan0"
         master_bin="" />

File: src/scara_4dof/urdf/scara_controller/robot_controller.macro.xacro (robot description, xacro)
@@ -39,5 +39,4 @@
         </visual>
     </link>
-    <!-- Adding link5 to fix the error -->
     <link name="${prefix}link5">
         <visual>
@@ -53,5 +52,5 @@
         <child link="${prefix}link1"/>
     </joint>
-    <joint name="${prefix}joint1" type="prismatic">
+    <joint name="${prefix}joint1" type="revolute">
         <parent link="${prefix}link1"/>
         <child link="${prefix}link2"/>

File: src/scara_4dof/urdf/scara_controller/robot_controller.ros2_control.xacro (robot description, xacro)
@@ -16,31 +16,19 @@
               <param name="master_bin">"${master_bin}"</param>
             </hardware>
-            <!-- Prismatic Joint -->
             <joint name="${prefix}joint1">
                 <param name="device_name">joint_1</param>
                 <state_interface name="position" />
-                <command_interface name="position" />
             </joint>
-            <!-- Revolute Joints -->
             <joint name="${prefix}joint2">
                 <param name="device_name">joint_2</param>
                 <state_interface name="position" />
-                <command_interface name="position" />
-                <state_interface name="velocity" />
-                <command_interface name="velocity" />
             </joint>
             <joint name="${prefix}joint3">
                 <param name="device_name">joint_3</param>
                 <state_interface name="position" />
-                <command_interface name="position" />
-                <state_interface name="velocity" />
-                <command_interface name="velocity" />
             </joint>
             <joint name="${prefix}joint4">
                 <param name="device_name">joint_4</param>
                 <state_interface name="position" />
-                <command_interface name="position" />
-                <state_interface name="velocity" />
-                <command_interface name="velocity" />
             </joint>
         </ros2_control>

File: src/scara_4dof/urdf/scara_controller/robot_controller.urdf.xacro (robot description, xacro)
@@ -1,10 +1,7 @@
 <?xml version="1.0"?>
 <robot xmlns:xacro="http://wiki.ros.org/xacro" name="test_robot">
-    <!-- Include the robot structure and control configuration macros -->
     <xacro:include filename="$(find scara_4dof)/urdf/scara_controller/robot_controller.macro.xacro"/>
     <xacro:include filename="$(find scara_4dof)/urdf/scara_controller/robot_controller.ros2_control.xacro"/>
-    <!-- Define the world link -->
     <link name="world" />
-    <!-- Invoke the macro to create the robot -->
     <xacro:robot_control_robot
         name="test_robot"
@@ -13,10 +10,9 @@
         <origin xyz="0 0 0" rpy="0 0 0" />
     </xacro:robot_control_robot>
-    <!-- Invoke the macro for ROS 2 control configuration -->
     <xacro:robot_control_control
         name="test_robot"
         prefix=""
-        bus_config="$(find scara_4dof)/config/scara_control/bus.yml"
-        master_config="$(find scara_4dof)/config/scara_control/master.dcf"
+        bus_config="$(find canopen_tests)/config/scara_4dof_control/bus.yml"
+        master_config="$(find canopen_tests)/config/scara_4dof_control/master.dcf"
         can_interface_name="vcan0"
         master_bin="" />
