Commit message: removed seperate scara control package.

File: src/canopen_tests/urdf/scara_controller/robot_controller.macro.xacro (robot description, xacro)
@@ -11,5 +11,5 @@
             <origin xyz="0 0 0" rpy="0 0 0"/>
             <geometry>
-                <cylinder radius="0.2" length="0.5"/>
+                <cylinder radius="0.2" length="0.01"/>
             </geometry>
         </visual>
@@ -52,8 +52,8 @@
         <child link="${prefix}link1"/>
     </joint>
-    <joint name="${prefix}joint1" type="revolute">
+    <joint name="${prefix}joint1" type="prismatic">
         <parent link="${prefix}link1"/>
         <child link="${prefix}link2"/>
-        <origin xyz="0 0 0.5" rpy="0 0 0"/>
+        <origin xyz="0 0 0.01" rpy="0 0 0"/>
         <axis xyz="0 1 0" />
         <limit lower="0" upper="0.1" effort="100.0" velocity="0.1"/>

File: src/canopen_tests/urdf/scara_controller/robot_controller.urdf.xacro (robot description, xacro)
@@ -8,5 +8,5 @@
         prefix=""
         parent="world">
-        <origin xyz="0 0 0" rpy="0 0 0" />
+        <origin xyz="0 0 1" rpy="1.57 0 0" />
     </xacro:robot_control_robot>
     <xacro:robot_control_control

Commit message: added third joint to urdf. and updated shell script to run inside docker.

File: src/canopen_tests/urdf/scara_controller/robot_controller.macro.xacro (robot description, xacro)
@@ -73,9 +73,16 @@
         <limit lower="${-2*pi}" upper="${2*pi}" effort="10.0" velocity="0.5"/>
     </joint>
-    <joint name="${prefix}joint4" type="fixed">
+    <joint name="${prefix}joint4" type="revolute">
+        <parent link="${prefix}link3"/>
+        <child link="${prefix}link4"/>
+        <origin xyz="0 0 0.5" rpy="0 0 0"/>
+        <axis xyz="0 1 0" />
+        <limit lower="${-2*pi}" upper="${2*pi}" effort="10.0" velocity="0.5"/>
+    </joint>
+    <joint name="${prefix}tool_joint" type="fixed">
         <parent link="${prefix}link4"/>
         <child link="${prefix}link5"/>
-        <origin xyz="0 0 0.5" rpy="0 0 0"/>
-        <axis xyz="0 1 0" />
+        <origin xyz="0 0 0.1" rpy="0 0 0"/>
+        <axis xyz="0 0 1" />
     </joint>
     </xacro:macro>
