Commit message: removed fourth joint

File: src/canopen_tests/urdf/scara_controller/robot_controller.ros2_control.xacro (robot description, xacro)
@@ -28,8 +28,8 @@
                 <state_interface name="position" />
             </joint>
-            <joint name="${prefix}joint4">
+            <!-- <joint name="${prefix}joint4">
                 <param name="device_name">joint_4</param>
                 <state_interface name="position" />
-            </joint>
+            </joint> -->
         </ros2_control>
     </xacro:macro>
